Commit message: testing a lot of stuff with rtabmap, robot localization, ros 2 control and nav2

File: description/lidar.xacro (robot description, xacro)
@@ -4,5 +4,5 @@
 		<parent link="chassis" />
 		<child link="laser_frame" />
-		<origin xyz="0 0 0.12" rpy="0 0 ${pi}" />
+		<origin xyz="0 0 0.2" rpy="0 0 ${pi}" />
 	</joint>
 	<link name="laser_frame">
@@ -31,5 +31,5 @@
 			</pose>
 			<visualize>
-				true
+				false
 			</visualize>
 			<update_rate>

File: description/robot.urdf.xacro (robot description, xacro)
@@ -4,3 +4,4 @@
     <xacro:include filename="gazebo_control.xacro"/>
     <xacro:include filename="lidar.xacro"/>
+    <xacro:include filename="depth_camera.xacro"/>
 </robot>
