Commit message: bugfixing

File: description/IMU.xacro (robot description, xacro)
@@ -4,10 +4,10 @@
         <parent link="chassis" />
         <child link="imu_frame" />
-        <origin xyz="0 0 0.2" rpy="0 0 0" />
+        <origin xyz="0 0 0.1" rpy="0 0 0" />
     </joint>
     <link name="imu_frame">
         <visual>
             <geometry>
-                <box size="0.1 0.1 0.05" />
+                <box size="0.01 0.01 0.001" />
             </geometry>
             <material name="blue" />
@@ -15,8 +15,8 @@
         <collision>
             <geometry>
-                <box size="0.1 0.1 0.05" />
+                <box size="0.01 0.01 0.001" />
             </geometry>
         </collision>
-        <xacro:inertial_box mass="0.1" size="0.1 0.1 0.05">
+        <xacro:inertial_box mass="0.01" x="0.01" y="0.01" z="0.001">
             <origin xyz="0 0 0" rpy="0 0 0" />
         </xacro:inertial_box>

File: description/depth_camera.xacro (robot description, xacro)
@@ -4,5 +4,5 @@
         <parent link="chassis"/>
         <child link="camera_link"/>
-        <origin xyz="0.305 0 0.08" rpy="0 0 0"/>
+        <origin xyz="${0.335/2} 0 0.08" rpy="0 0 0"/>
     </joint>
     <link name="camera_link">

File: description/robot.urdf.xacro (robot description, xacro)
@@ -2,5 +2,5 @@
 <robot xmlns:xacro="http://www.ros.org/wiki/xacro"  name="robot">
     <xacro:arg name="use_ros2_control" default="true"/>
-    <xacro:arg name="sim_mode" default="false"/>
+    <xacro:arg name="sim_mode" default="true"/>
     <xacro:include filename="robot_core.xacro" />
     <xacro:if value="$(arg use_ros2_control)">

File: description/ros2_control.xacro (robot description, xacro)
@@ -54,5 +54,5 @@
                 <plugin>gazebo_ros2_control/GazeboSystem</plugin>
             </hardware>
-            <joint name="left_wheel_joint">
+            <joint name="front_left_wheel_joint">
                 <command_interface name="velocity">
                     <param name="min">-10</param>
@@ -62,5 +62,21 @@
                 <state_interface name="position"/>
             </joint>
-            <joint name="right_wheel_joint">
+            <joint name="front_right_wheel_joint">
+                <command_interface name="velocity">
+                    <param name="min">-10</param>
+                    <param name="max">10</param>
+                </command_interface>
+                <state_interface name="velocity"/>
+                <state_interface name="position"/>
+            </joint>
+            <joint name="back_left_wheel_joint">
+                <command_interface name="velocity">
+                    <param name="min">-10</param>
+                    <param name="max">10</param>
+                </command_interface>
+                <state_interface name="velocity"/>
+                <state_interface name="position"/>
+            </joint>
+            <joint name="back_right_wheel_joint">
                 <command_interface name="velocity">
                     <param name="min">-10</param>
