Commit message: update urdf

File: description/gazebo_control.xacro (robot description, xacro)
@@ -9,8 +9,8 @@
         <right_joint>front_right_wheel_joint</right_joint>
         <right_joint>back_right_wheel_joint</right_joint>
-        <wheel_separation>0.35</wheel_separation>
-        <wheel_diameter>0.0889</wheel_diameter>
-        <wheel_separation>0.35</wheel_separation>
-        <wheel_diameter>0.0889</wheel_diameter>
+        <wheel_separation>0.19685</wheel_separation>
+        <wheel_diameter>0.06985</wheel_diameter>
+        <wheel_separation>0.19685</wheel_separation>
+        <wheel_diameter>0.06985</wheel_diameter>
         <!-- Limits -->
         <max_wheel_torque>200</max_wheel_torque>

File: description/lidar.xacro (robot description, xacro)
@@ -4,10 +4,10 @@
 		<parent link="chassis" />
 		<child link="laser_frame" />
-		<origin xyz="0 0 0.2" rpy="0 0 ${pi}" />
+		<origin xyz="0 0 0.17145" rpy="0 0 ${-pi/2}" />
 	</joint>
 	<link name="laser_frame">
 		<visual>
 			<geometry>
-				<cylinder radius="0.05" length="0.04" />
+				<cylinder radius="0.03175" length="0.0381" />
 			</geometry>
 			<material name="red" />
@@ -15,9 +15,9 @@
 		<collision>
 			<geometry>
-				<cylinder radius="0.05" length="0.04" />
+				<cylinder radius="0.03175" length="0.0381" />
 			</geometry>
 		</collision>
-		<xacro:inertial_cylinder mass="0.1" length="0.04" radius="0.05">
-			<origin xyz="0 0 0" rpy="0 0 ${pi}" />
+		<xacro:inertial_cylinder mass="0.1" length="0.0381" radius="0.03175">
+			<origin xyz="0 0 0" rpy="0 0 ${-pi/2}" />
 		</xacro:inertial_cylinder>
 	</link>

File: description/robot_core.xacro (robot description, xacro)
@@ -2,14 +2,14 @@
 <robot xmlns:xacro="http://www.ros.org/wiki/xacro">
     <xacro:include filename="inertial_macros.xacro"/>
-    <xacro:property name="chassis_length" value="0.335"/>
-    <xacro:property name="chassis_width" value="0.265"/>
-    <xacro:property name="chassis_height" value="0.138"/>
+    <xacro:property name="chassis_length" value="0.254"/>
+    <xacro:property name="chassis_width" value="0.1524"/>
+    <xacro:property name="chassis_height" value="0.1651"/>
     <xacro:property name="chassis_mass" value="1.0"/>
-    <xacro:property name="wheel_radius" value="0.04445"/>
-    <xacro:property name="wheel_thickness" value="0.026"/>
+    <xacro:property name="wheel_radius" value="0.034925"/>
+    <xacro:property name="wheel_thickness" value="0.028575"/>
     <xacro:property name="wheel_mass" value="0.05"/>
-    <xacro:property name="wheel_offset_x" value="0.05"/>
-    <xacro:property name="wheel_offset_y" value="0.1485"/>
-    <xacro:property name="wheel_offset_z" value="0.01"/>
+    <xacro:property name="wheel_offset_x" value="0.0762"/>
+    <xacro:property name="wheel_offset_y" value="0.098425"/>
+    <xacro:property name="wheel_offset_z" value="0.01905"/>
     <material name="white">
         <color rgba="1 1 1 1"/>
