Commit message: Update robot_core.xacro

File: description/robot_core.xacro (robot description, xacro)
@@ -9,5 +9,5 @@
     <xacro:property name="wheel_thickness" value="0.028575"/>
     <xacro:property name="wheel_mass" value="0.05"/>
-    <xacro:property name="wheel_offset_x" value="0.0762"/>
+    <xacro:property name="wheel_offset_x" value="0.0677"/>
     <xacro:property name="wheel_offset_y" value="0.098425"/>
     <xacro:property name="wheel_offset_z" value="0.01905"/>

Commit message: Update robot_core.xacro

File: description/robot_core.xacro (robot description, xacro)
@@ -9,5 +9,5 @@
     <xacro:property name="wheel_thickness" value="0.028575"/>
     <xacro:property name="wheel_mass" value="0.05"/>
-    <xacro:property name="wheel_offset_x" value="0.0677"/>
+    <xacro:property name="wheel_offset_x" value="0.067691"/>
     <xacro:property name="wheel_offset_y" value="0.098425"/>
     <xacro:property name="wheel_offset_z" value="0.01905"/>

Commit message: Update robot_core.xacro

File: description/robot_core.xacro (robot description, xacro)
@@ -3,5 +3,5 @@
     <xacro:include filename="inertial_macros.xacro"/>
     <xacro:property name="chassis_length" value="0.254"/>
-    <xacro:property name="chassis_width" value="0.1524"/>
+    <xacro:property name="chassis_width" value="0.149225"/>
     <xacro:property name="chassis_height" value="0.1651"/>
     <xacro:property name="chassis_mass" value="1.0"/>

Commit message: trying to fix gazebo wheel drift issue?

File: description/robot_core.xacro (robot description, xacro)
@@ -11,5 +11,5 @@
     <xacro:property name="wheel_offset_x" value="0.0762"/>
     <xacro:property name="wheel_offset_y" value="0.098425"/>
-    <xacro:property name="wheel_offset_z" value="0.01905"/>
+    <xacro:property name="wheel_offset_z" value="-0.01905"/>
     <material name="white">
         <color rgba="1 1 1 1"/>
@@ -71,4 +71,6 @@
         <origin xyz="${wheel_offset_x} ${-wheel_offset_y} 0" rpy="${pi/2} 0 0"/>
         <axis xyz="0 0 -1"/>
+        <limit effort="10000" velocity="1000"/>
+        <dynamics damping="1.0" friction="1.0"/>
     </joint>
     <link name="front_left_wheel">
@@ -97,4 +99,6 @@
         <origin xyz="${-wheel_offset_x} ${-wheel_offset_y} 0" rpy="${pi/2} 0 0"/>
         <axis xyz="0 0 -1"/>
+        <limit effort="10000" velocity="1000"/>
+        <dynamics damping="1.0" friction="1.0"/>
     </joint>
     <link name="back_left_wheel">
@@ -123,4 +127,6 @@
         <origin xyz="${wheel_offset_x} ${wheel_offset_y} 0" rpy="-${pi/2} 0 0"/>
         <axis xyz="0 0 1"/>
+        <limit effort="10000" velocity="1000"/>
+        <dynamics damping="1.0" friction="1.0"/>
     </joint>
     <link name="front_right_wheel">
@@ -149,4 +155,6 @@
         <origin xyz="${-wheel_offset_x} ${wheel_offset_y} 0" rpy="-${pi/2} 0 0"/>
         <axis xyz="0 0 1"/>
+        <limit effort="10000" velocity="1000"/>
+        <dynamics damping="1.0" friction="1.0"/>
     </joint>
     <link name="back_right_wheel">
@@ -159,5 +167,5 @@
         <collision>
             <geometry>
-                <cylinder radius="${wheel_radius}" length="${wheel_thickness}"/>
+                <sphere radius="${wheel_radius}"/>
             </geometry>
         </collision>

Commit message: Update robot_core.xacro

File: description/robot_core.xacro (robot description, xacro)
@@ -2,5 +2,5 @@
 <robot xmlns:xacro="http://www.ros.org/wiki/xacro">
     <xacro:include filename="inertial_macros.xacro"/>
-    <xacro:property name="chassis_length" value="0.254"/>
+    <xacro:property name="chassis_length" value="0.24455"/>
     <xacro:property name="chassis_width" value="0.149225"/>
     <xacro:property name="chassis_height" value="0.1651"/>

Commit message: Update robot_core.xacro

File: description/robot_core.xacro (robot description, xacro)
@@ -9,7 +9,7 @@
     <xacro:property name="wheel_thickness" value="0.028575"/>
     <xacro:property name="wheel_mass" value="0.05"/>
-    <xacro:property name="wheel_offset_x" value="0.067691"/>
-    <xacro:property name="wheel_offset_y" value="0.098425"/>
-    <xacro:property name="wheel_offset_z" value="-0.01905"/>
+    <xacro:property name="wheel_offset_x" value="0.1016"/>
+    <xacro:property name="wheel_offset_y" value="0.0993"/>
+    <xacro:property name="wheel_offset_z" value="0.0150241"/>
     <material name="white">
         <color rgba="1 1 1 1"/>

Commit message: Update robot_core.xacro

File: description/robot_core.xacro (robot description, xacro)
@@ -5,5 +5,5 @@
     <xacro:property name="chassis_width" value="0.149225"/>
     <xacro:property name="chassis_height" value="0.1651"/>
-    <xacro:property name="chassis_mass" value="1.0"/>
+    <xacro:property name="chassis_mass" value="3.40194"/>
     <xacro:property name="wheel_radius" value="0.034925"/>
     <xacro:property name="wheel_thickness" value="0.028575"/>

Commit message: update dimentions

File: description/robot_core.xacro (robot description, xacro)
@@ -11,5 +11,5 @@
     <xacro:property name="wheel_offset_x" value="0.1016"/>
     <xacro:property name="wheel_offset_y" value="0.0993"/>
-    <xacro:property name="wheel_offset_z" value="0.0150241"/>
+    <xacro:property name="wheel_offset_z" value="-0.0150241"/>
     <material name="white">
         <color rgba="1 1 1 1"/>
