Commit message: untested new gazebo

File: description/depth_camera.xacro (robot description, xacro)
@@ -11,5 +11,5 @@
                 <box size="0.010 0.03 0.03"/>
             </geometry>
-            <material name="red"/>
+            <material name="black"/>
         </visual>
     </link>
@@ -21,5 +21,5 @@
     <link name="camera_link_optical"></link>
 <gazebo reference="camera_link">
-    <material>Gazebo/Red</material>
+    <material>Gazebo/Black</material>
     <sensor name="camera" type="depth">
         <pose>0 0 0 0 0 0</pose>
@@ -39,9 +39,6 @@
             </clip>
         </camera>
-        <plugin name="camera_controller" filename="libgazebo_ros_camera.so">
-            <frame_name>camera_link_optical</frame_name>
-            <min_depth>0.1</min_depth> <!-- Minimum depth sensing limit for the D450 -->
-            <max_depth>10.0</max_depth> <!-- Maximum depth sensing limit for the D450 -->
-        </plugin>
+        <topic>camera/image_raw</topic>
+        <gz_frame_id>camera_link_optical</gz_frame_id>
     </sensor>
 </gazebo>

File: description/gazebo_control.xacro (robot description, xacro)
@@ -2,24 +2,33 @@
 <robot xmlns:xacro="http://www.ros.org/wiki/xacro">
     <gazebo>
-        <plugin name='diff_drive' filename='libgazebo_ros_diff_drive.so'>
-        <num_wheel_pairs>2</num_wheel_pairs>
-        <!-- Wheel Information -->
-        <left_joint>front_left_wheel_joint</left_joint>
-        <left_joint>back_left_wheel_joint</left_joint>
-        <right_joint>front_right_wheel_joint</right_joint>
-        <right_joint>back_right_wheel_joint</right_joint>
-        <wheel_separation>0.19685</wheel_separation>
-        <wheel_diameter>0.06985</wheel_diameter>
-        <wheel_separation>0.19685</wheel_separation>
-        <wheel_diameter>0.06985</wheel_diameter>
-        <!-- Limits -->
-        <max_wheel_torque>200</max_wheel_torque>
-        <max_wheel_acceleration>10.0</max_wheel_acceleration>
-        <!-- Output -->
-        <odometry_frame>odom</odometry_frame>
-        <robot_base_frame>base_link</robot_base_frame>
-        <publish_odom>true</publish_odom>
-        <publish_odom_tf>true</publish_odom_tf>
-        <publish_wheel_tf>true</publish_wheel_tf>
+        <plugin name="gz::sim::systems::DiffDrive" filename="gz-sim-diff-drive-system">
+            <num_wheel_pairs>2</num_wheel_pairs>
+            <!-- Wheel Information -->
+            <left_joint>front_left_wheel_joint</left_joint>
+            <left_joint>back_left_wheel_joint</left_joint>
+            <right_joint>front_right_wheel_joint</right_joint>
+            <right_joint>back_right_wheel_joint</right_joint>
+            <wheel_separation>0.19685</wheel_separation>
+            <wheel_radius>0.034925</wheel_radius>
+            <wheel_separation>0.19685</wheel_separation>
+            <wheel_radius>0.034925</wheel_radius>
+            <!-- Limits -->
+            <max_linear_acceleration>0.33</max_linear_acceleration>
+            <!-- Input -->
+            <topic>cmd_vel</topic>
+            <!-- Output -->
+            <frame_id>odom</frame_id>
+            <child_frame_id>base_link</child_frame_id>
+            <odom_topic>odom</odom_topic>
+            <odom_publisher_frequency>30</odom_publisher_frequency>
+            <tf_topic>/tf</tf_topic>
+        </plugin>
+        <plugin filename="gz-sim-joint-state-publisher-system"
+            name="gz::sim::systems::JointStatePublisher">
+            <topic>joint_states</topic>
+            <joint_name>front_left_wheel_joint</joint_name>
+            <joint_name>front_right_wheel_joint</joint_name>
+            <joint_name>back_left_wheel_joint</joint_name>
+            <joint_name>back_right_wheel_joint</joint_name>
         </plugin>
     </gazebo>

File: description/lidar.xacro (robot description, xacro)
@@ -22,55 +22,26 @@
 		</xacro:inertial_cylinder>
 	</link>
-	<gazebo reference="laser_frame">
-		<material>
-			Gazebo/Red
-		</material>
-		<sensor name="laser" type="ray">
-			<pose>
-				0 0 0 0 0 0
-			</pose>
-			<visualize>
-				false
-			</visualize>
-			<update_rate>
-				10
-			</update_rate>
-			<ray>
-				<scan>
-					<horizontal>
-						<samples>
-							360
-						</samples>
-						<min_angle>
-							3.14159
-						</min_angle>
-						<max_angle>
-							-3.14159
-						</max_angle>
-					</horizontal>
-				</scan>
-				<range>
-					<min>
-						0.3
-					</min>
-					<max>
-						12
-					</max>
-				</range>
-			</ray>
-			<plugin name="laser_controller" filename="libgazebo_ros_ray_sensor.so">
-				<ros>
-					<argument>
-						~/out:=scan
-					</argument>
-				</ros>
-				<output_type>
-					sensor_msgs/LaserScan
-				</output_type>
-				<frame_name>
-					laser_frame
-				</frame_name>
-			</plugin>
-		</sensor>
-	</gazebo>
+    <gazebo reference="laser_frame">
+        <material>Gazebo/Black</material>
+        <sensor name="laser" type="gpu_lidar">
+            <pose> 0 0 0 0 0 0 </pose>
+            <visualize>false</visualize>
+            <update_rate>10</update_rate>
+            <lidar>
+                <scan>
+                    <horizontal>
+                        <samples>360</samples>
+                        <min_angle>-3.14</min_angle>
+                        <max_angle>3.14</max_angle>
+                    </horizontal>
+                </scan>
+                <range>
+                    <min>0.3</min>
+                    <max>12</max>
+                </range>
+            </lidar>
+            <topic>scan</topic>
+            <gz_frame_id>laser_frame</gz_frame_id>
+        </sensor>
+    </gazebo>
 </robot>

File: description/ros2_control.xacro (robot description, xacro)
@@ -56,5 +56,5 @@
         <ros2_control name="GazeboSystem" type="system">
             <hardware>
-                <plugin>gazebo_ros2_control/GazeboSystem</plugin>
+                <plugin>gz_ros2_control/GazeboSimSystem</plugin>
             </hardware>
             <joint name="front_left_wheel_joint">
@@ -93,5 +93,5 @@
     </xacro:if>
     <gazebo>
-        <plugin name="gazebo_ros2_control" filename="libgazebo_ros2_control.so">
+        <plugin name="gz_ros2_control::GazeboSimROS2ControlPlugin" filename="libgz_ros2_control-system.so">
             <parameters>$(find my_bot)/config/my_controllers.yaml</parameters>
             <parameters>$(find my_bot)/config/gaz_ros2_ctl_use_sim.yaml</parameters>
